File: Yaesu/Yaesu.kicad_sch (KiCad schematic)
At the start: 15 parts, among them J1 OHIS RJ45, J2 Yaesu HF RJ45 Mic, J3 Yaesu HF GX16-8P Mic, J4 Headphone In, J5 Speaker In, J6 Yaesu Mobile Mic In

Commit message: Yaesu mic pinout references.  #1
Connections:
- net Earth renamed Shield
Other:
- note added: "Tie all "Shield"s to metalic case. DO NOT TIE TO GROUND!"
- moved on the sheet: J3, J4, J5, J6, JP1, R5, R6
