File: Kenwood/Kenwood.kicad_sch (KiCad schematic)
At the start: 10 parts, among them J1 OHIS RJ45, J2 Kenwood RJ45 Mic, J3 Kenwood GX16-8P Mic, J4 Headphone In

Commit message: Kenwood laid out more similarly to the User Adapter. #1
Parts:
- removed J4: Headphone In, symbol Connector_Audio:AudioJack3_Ground_Switch
- added C3, C4: 10uF, Capacitor_SMD:C_1206_3216Metric, symbol Device:C_Small
- added G1: Board_Artwork, OHIS:Logo_OHIS_Small, symbol Smitty:Board_Artwork
- added H1, H2, H3, H4: MountingHole_Pad, MountingHole:MountingHole_3.2mm_M3_Pad, symbol Mechanical:MountingHole_Pad
- added J4: Headphone In, Libraries:Conn_3.5mm-PJ-393_SMT-C668609_TH-C145811, symbol Smitty:AudioJack4_SwitchTR1R2S
- added J6: Speaker Input Config, Connector_PinHeader_2.54mm:PinHeader_2x04_P2.54mm_Horizontal, symbol Connector_Generic:Conn_02x04_Odd_Even
- added R10, R12: 1k, Resistor_SMD:R_1206_3216Metric, symbol Device:R_Small
- added R11: 6.2k, Resistor_SMD:R_1206_3216Metric, symbol Device:R_Small
- added R5, R7, R9: 100R, Resistor_SMD:R_1206_3216Metric, symbol Device:R_Small
- added R6, R8: 100R, Resistor_THT:R_Axial_DIN0207_L6.3mm_D2.5mm_P7.62mm_Horizontal, symbol Device:R_Small
- C1, C2: footprint (none) -> Capacitor_THT:C_Disc_D4.7mm_W2.5mm_P5.00mm
- J1: footprint (none) -> Connector_RJ:RJ45_Amphenol_RJHSE538X
- J2: footprint (none) -> Connector_RJ:RJ45_Amphenol_RJHSE538X; symbol Connector:RJ45_Shielded -> Connector:RJ45_LED_Shielded
- J3: now not fitted; now left out of the parts list
- R1, R2, R3, R4: footprint (none) -> Resistor_THT:R_Axial_DIN0207_L6.3mm_D2.5mm_P7.62mm_Horizontal
Connections:
- net +8v 10mA: now also R11.1, R12.1
- net AF Out: now also J4.R1N, J4.TN
- net HP Gnd: now also J4.R2, J4.S
- net HP Left: now also J6.7 (Pin_7), R5.1, R6.1
- net HP Right: now also J6.5 (Pin_5), R7.1, R8.2
- net Mic Gnd: now also R9.2
- net Mic+: now also C4.2
- net OHIS Mic+: now also C3.2, R11.2
- net Power Gnd: now also J4.SN
- net Shield: now also H1.1, H2.1, H3.1, H4.1
- net at J1.10, R1.2: now also R12.2
- net at C2.1, R2.2, R3.1: now also C4.1, R10.2, R9.1
- net at C1.1, R2.1: now also C3.1, R10.1
- new net: J4.R1, J6.1 (Pin_1)
- new net: J6.2 (Pin_2), J6.4 (Pin_4), J6.6 (Pin_6), R7.2, R8.1
- new net: J4.T, J6.3 (Pin_3), J6.8 (Pin_8), R5.2, R6.2
- no-connect marks 3 -> 8
Other:
- note added: "Jumper: Headphone No Jumper: Speaker"
- note added: "Mono Source"
- note added: "Overrides AF Out from Mic connector."
- note added: "Stereo Source"
- moved on the sheet: C1, C2, R1, R4
