File: BaseBoard/BaseBoard.kicad_pcb (KiCad board)
At the start: 2 copper layers, 74.3 x 30.5 mm, 22 parts, among them J1 OHIS RJ45, J2 Radio Board, J3 Dynamic/Electret, J6 Speaker Input Config

Commit message: Happy with BaseBoard and Icom-RJ45. Working on Icom-GX16 #1
Parts:
- added G2: Board_Artwork, OHIS:Logo_OHIS_Medium, F.Cu at (146.1, 66.7)
- G1: footprint OHIS:Logo_OHIS_Small -> OHIS:Logo_OHIS_Medium
- moved G1 46.1 mm to (146.1, 90.8)
- moved RV1 5.61 mm to (102.2, 66.7), turned to -90 degrees
Routing:
- net Net-(C1-Pad1): track 3.57 -> 9.68 mm
- net Radio Mic Gnd: track 87.3 -> 93.3 mm
- net Net-(C2-Pad1): track 5.29 -> 2.94 mm
- net Radio +V: track 24.9 -> 26.0 mm
- net Shield: vias 0 -> 190
Other:
- board text added: "Dyn"
- board text added: "Elec"
- board text added: "JLCJLCJLCJLC"
- board text added: "Mic Level"
- board text added: "Mic:"
- board text added: "Mono"
- board text added: "OHIS Radio Adapter v1.0a 2024 CC-BY OHIS-WG ohis.org"
- board text added: "Phones"
- board text added: "Radio Board Here"
- board text added: "Spkr"
- board text added: "Spkr/ Phones:"
- board text added: "Stereo"

Commit message: Updated BOM parts, among other things. Sorry, it's been a while. #1
Parts:
- removed RV1: 1k, Potentiometer_THT:Potentiometer_Piher_PT-6-H_Horizontal
- added BOM1: M3 6mm SS screw, Libraries:BOM_Item, F.Cu at (109.1, 65.8)
- added BOM10: M3 14mm brass standoff, Libraries:BOM_Item, F.Cu at (107.6, 68.8)
- added BOM11: M3 3mm ABS standoff, Libraries:BOM_Item, F.Cu at (106.1, 68.8)
- added BOM12: M3 10mm SS screw, Libraries:BOM_Item, F.Cu at (104.6, 68.8)
- added BOM13: M3 6mm SS screw, Libraries:BOM_Item, F.Cu at (109.1, 70.3)
- added BOM14: M3 14mm brass standoff, Libraries:BOM_Item, F.Cu at (107.6, 70.3)
- added BOM15: M3 3mm ABS standoff, Libraries:BOM_Item, F.Cu at (106.1, 70.3)
- added BOM16: M3 10mm SS screw, Libraries:BOM_Item, F.Cu at (104.6, 70.3)
- added BOM17: M3 6mm SS screw, Libraries:BOM_Item, F.Cu at (109.1, 71.8)
- added BOM18: M3 14mm brass standoff, Libraries:BOM_Item, F.Cu at (107.6, 71.8)
- added BOM19: M3 3mm ABS standoff, Libraries:BOM_Item, F.Cu at (106.1, 71.8)
- added BOM2: Top Board, Libraries:BOM_Item, F.Cu at (107.6, 65.8)
- added BOM20: .1" Jumper, Libraries:BOM_Item, F.Cu at (104.6, 71.8)
- added BOM21: .1" Jumper, Libraries:BOM_Item, F.Cu at (109.1, 73.3)
- added BOM22: .1" Jumper, Libraries:BOM_Item, F.Cu at (107.6, 73.3)
- added BOM23: .1" Jumper, Libraries:BOM_Item, F.Cu at (106.1, 73.3)
- added BOM24: .1" Jumper, Libraries:BOM_Item, F.Cu at (104.6, 73.3)
- added BOM3: M3 14mm brass standoff, Libraries:BOM_Item, F.Cu at (106.1, 65.8)
- added BOM4: Main Board, Libraries:BOM_Item, F.Cu at (104.6, 65.8)
- added BOM5: Bottom Board, Libraries:BOM_Item, F.Cu at (109.1, 67.3)
- added BOM6: M3 10mm SS screw, Libraries:BOM_Item, F.Cu at (107.6, 67.3)
- added BOM7: M3 3mm ABS standoff, Libraries:BOM_Item, F.Cu at (106.1, 67.3)
- added BOM8: M3 10mm SS screw, Libraries:BOM_Item, F.Cu at (104.6, 67.3)
- added BOM9: M3 6mm SS screw, Libraries:BOM_Item, F.Cu at (109.1, 68.8)
- added RV2: 1k, Potentiometer_THT:Potentiometer_Piher_PT-6-H_Horizontal, F.Cu at (102.2, 66.7)
Other:
- board text added: "OHIS Radio Adapter v1.0b 2024 CC-BY OHIS-WG ohis.org"
- board text removed: "OHIS Radio Adapter v1.0a 2024 CC-BY OHIS-WG ohis.org"
